File: shield/shield.kicad_pcb (KiCad board)
At the start: 2 copper layers, 17.8 x 33 mm, 12 parts, among them J1 Booster, J2 Battery, P1 Digital, P2 COM, P3 ADC, P4 Analog, P5 ADC, U1 RFM69HW

Commit message: hi
Parts:
- removed P1: Digital, Socket_Arduino_Pro_Mini:Socket_Strip_Arduino_1x12
- removed P2: COM, Socket_Arduino_Pro_Mini:Socket_Strip_Arduino_1x06
- removed P3, P5: ADC, Socket_Arduino_Pro_Mini:Socket_Strip_Arduino_1x02
- removed P4: Analog, Socket_Arduino_Pro_Mini:Socket_Strip_Arduino_1x12
- removed U1: RFM69HW, RF_Module:HOPERF_RFM69HW
- added ?: , Connector_PinHeader_2.54mm:PinHeader_1x02_P2.54mm_Vertical, F.Cu at (117.2, 91.4)
- added ?: , Connector_PinHeader_2.54mm:PinHeader_1x02_P2.54mm_Vertical, F.Cu at (117.2, 94.0)
- added REF**: HOPERF_RFM69HW, RF_Module:HOPERF_RFM69HW, F.Cu at (103.6, 67.8)
- added REF**: ArduinoProMini, footprints:pro_mini_rfmshield, F.Cu at (102.1, 77.0)
- C2: moved to B.Cu
- moved J2 90.2 mm to (113.8, 133.4), turned to 90 degrees
- moved C2 57.1 mm to (121.1, 105.7), turned to 180 degrees
Connections:
- net /A0 renamed Net-(C1-Pad1)
- net GND renamed Net-(C1-Pad2)
Routing:
- net (no net): track 0.00 -> 83.6 mm
- net Net-(C1-Pad2): track 0.00 -> 27.7 mm
Other:
- board outline removed
- board text removed: "1"

Commit message: pre holiday commit
Parts:
- removed ? (x2): , Connector_PinHeader_2.54mm:PinHeader_1x02_P2.54mm_Vertical
- removed REF**: HOPERF_RFM69HW, RF_Module:HOPERF_RFM69HW
- removed REF**: ArduinoProMini, footprints:pro_mini_rfmshield
- added ProMini1: rfmshield_pro_mini_pins, footprints:pro_mini_rfmshield, F.Cu at (102.9, 75.6)
- added RFM69HW: RFM69HW, RF_Module:HOPERF_RFM69HW, F.Cu at (104.8, 66.0)
- added SCL: SCL Breakout, Connector_PinHeader_2.54mm:PinHeader_1x02_P2.54mm_Vertical, B.Cu at (98.6, 87.1)
- added SDA: SDA Breakout, Connector_PinHeader_2.54mm:PinHeader_1x02_P2.54mm_Vertical, B.Cu at (102.1, 87.1)
- Bat: renamed from J2; footprint Connector_PinHeader_2.54mm:PinHeader_1x03_P2.54mm_Horizontal -> Connector_PinHeader_2.54mm:PinHeader_1x02_P2.54mm_Vertical
- Booster: renamed from J1; value Booster -> Booster Pins; footprint Connector_PinHeader_2.54mm:PinHeader_1x02_P2.54mm_Horizontal -> Connector_PinHeader_2.54mm:PinHeader_1x03_P2.54mm_Vertical
- C1: value C Voltage Divider -> Volt Div; footprint Capacitor_THT:C_Rect_L7.0mm_W3.5mm_P2.50mm_P5.00mm -> Capacitor_THT:CP_Radial_D6.3mm_P2.50mm
- C2: footprint Capacitor_THT:C_Rect_L7.0mm_W3.5mm_P2.50mm_P5.00mm -> Capacitor_THT:CP_Radial_D6.3mm_P2.50mm; moved to F.Cu
- moved R2 94.3 mm to (99.1, 95.2), turned to -90 degrees
- moved C1 93.7 mm to (96.5, 110.5)
- moved R1 86.1 mm to (96.5, 95.2), turned to -90 degrees
- moved Booster 83.0 mm to (104.2, 95.9), turned to 90 degrees
- moved Bat 25.0 mm to (104.2, 110.2)
- moved C2 17.2 mm to (104.2, 102.2), turned to 0 degrees
Connections:
- net Net-(C1-Pad2) renamed GND
- Bat pad 1: /+ -> +3V3
- R1 pad 1: /+ -> +3V3
Routing:
- net (no net): track 83.6 -> 0.00 mm
- net GND: track 27.7 -> 76.2 mm
- net Net-(C2-Pad1): track 0.00 -> 45.5 mm
- net Net-(C1-Pad1): track 0.00 -> 41.5 mm
- net +3V3: track 0.00 -> 32.0 mm
- net Net-(RFM69HW1-Pad12): track 0.00 -> 16.6 mm
- net Net-(RFM69HW1-Pad13): track 0.00 -> 13.3 mm
- net Net-(RFM69HW1-Pad2): track 0.00 -> 12.9 mm
- net Net-(ProMini1-PadSDA): track 0.00 -> 10.8 mm
- net Net-(RFM69HW1-Pad14): track 0.00 -> 9.90 mm
- net Net-(RFM69HW1-Pad15): track 0.00 -> 7.15 mm
- net Net-(ProMini1-PadSCL): track 0.00 -> 6.80 mm
Other:
- board outline added: 19.8 x 62 mm
- board text added: "+"
- board text added: "-"
- board text added: "GND"
- board text added: "NSS"
- board text added: "in"
- board text added: "out"

Commit message: v1-pre renice
Parts:
- removed SCL: SCL Breakout, Connector_PinHeader_2.54mm:PinHeader_1x02_P2.54mm_Vertical
- removed SDA: SDA Breakout, Connector_PinHeader_2.54mm:PinHeader_1x02_P2.54mm_Vertical
- added GND: Conn_01x03_Female, Connector_PinHeader_2.54mm:PinHeader_1x03_P2.54mm_Vertical, F.Cu at (99.6, 84.8)
- C1: value Volt Div -> C Voltage Divider
- moved C1 13.6 mm to (109.7, 107.2), turned to 90 degrees
- moved J2 12.2 mm to (109.2, 99.1), turned to 180 degrees
- moved R1 12.1 mm to (94.5, 107.2), turned to 0 degrees
- moved R2 10.5 mm to (94.5, 104.6), turned to 0 degrees
- moved C2 7.87 mm to (97.0, 99.1), turned to 90 degrees
- moved J1 4.22 mm to (103.6, 100.1), turned to 180 degrees
- renumbered Booster to J1, Bat to J2, RFM69HW to RFM69HW1
Connections:
- ProMini1 pad GND2: unconnected-(ProMini1-PadGND2) -> Net-(J3-Pad1)
- ProMini1 pad SCL: Net-(ProMini1-PadSCL) -> unconnected-(ProMini1-PadSCL)
- ProMini1 pad SDA: Net-(ProMini1-PadSDA) -> unconnected-(ProMini1-PadSDA)
Routing:
- net Net-(C2-Pad1): track 45.5 -> 59.6 mm
- net Net-(ProMini1-PadSDA): track 10.8 -> 0.00 mm
- net Net-(J3-Pad1): track 0.00 -> 9.56 mm
- net Net-(C1-Pad1): track 41.5 -> 50.7 mm
- net +3V3: track 32.0 -> 23.3 mm
- net Net-(ProMini1-PadSCL): track 6.80 -> 0.00 mm
- net GND: track 76.2 -> 72.8 mm
Other:
- board size 19.8 x 62 mm -> 19.8 x 55.4 mm

Commit message: v1
Parts:
- moved GND 1.02 mm to (99.6, 83.8)
- renumbered J2 to Battery, J1 to Booster, RFM69HW1 to RFM69HW
Routing:
- net Net-(J3-Pad1): track 9.56 -> 10.2 mm
Other:
- board text added: "Pro Mini Header here"
- board text added: "Vin"
- board text added: "Vout"
- board text removed: "in"
- board text removed: "out"
Changed lines of the file:
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@@
     (property "Sheetname" "")
     (attr smd)
-    (fp_text reference "RFM69HW1" (at 0 -0.127 90) (layer "F.SilkS")
+    (fp_text reference "RFM69HW" (at 0 -0.127 90) (layer "F.SilkS")
       (effects (font (size 1 1) (thickness 0.15)))
     )
@@
     (property "Sheetname" "")
     (attr through_hole)
-    (fp_text reference "J1" (at -2.032 2.525 90) (layer "F.SilkS")
+    (fp_text reference "Booster" (at -2.54 2.525 90) (layer "F.SilkS")
       (effects (font (size 1 1) (thickness 0.15)))
     )
@@
     (property "Sheetname" "")
     (attr through_hole)
-    (fp_text reference "J2" (at -3.556 1.27 90) (layer "F.SilkS")
+    (fp_text reference "Battery" (at -3.048 1.27 90) (layer "F.SilkS")
       (effects (font (size 1 1) (thickness 0.15)))
     )
@@
   )
   (footprint "Connector_PinHeader_2.54mm:PinHeader_1x03_P2.54mm_Vertical" (layer "F.Cu")
-    (at 99.568 84.836)
+    (at 99.568 83.82)
     (descr "Through hole straight pin header, 1x03, 2.54mm pitch, single row")
     (tags "Through hole pin header THT 1x03 2.54mm single row")
@@
     (property "Sheetname" "")
     (attr through_hole)
-    (fp_text reference "GND" (at 0 -2.33) (layer "F.SilkS")
+    (fp_text reference "GND" (at 2.54 2.54 90) (layer "F.SilkS")
       (effects (font (size 1 1) (thickness 0.15)))
     )
@@
   (gr_line (start 113.284 54.356) (end 113.284 109.728) (layer "Edge.Cuts") (width 0.1))
   (gr_line (start 113.284 109.728) (end 93.472 109.728) (layer "Edge.Cuts") (width 0.1))
+  (gr_text "Pro Mini Header here" (at 103.632 91.948) (layer "F.SilkS")
+    (effects (font (size 0.5 0.5) (thickness 0.125)))
+  )
   (gr_text "GND\n" (at 101.6 97.536 90) (layer "F.SilkS")
     (effects (font (size 0.5 0.5) (thickness 0.125)))
@@
     (effects (font (size 1 1) (thickness 0.15)))
   )
-  (gr_text "in" (at 101.6 94.996 90) (layer "F.SilkS")
+  (gr_text "Vin" (at 101.6 94.996 90) (layer "F.SilkS")
     (effects (font (size 0.5 0.5) (thickness 0.125)))
   )
@@
     (effects (font (size 1 1) (thickness 0.15)))
   )
-  (gr_text "out" (at 101.6 100.076 90) (layer "F.SilkS")
+  (gr_text "Vout" (at 101.6 100.076 90) (layer "F.SilkS")
     (effects (font (size 0.5 0.5) (thickness 0.125)))
   )
@@
   (segment (start 103.632 94.981) (end 95.612511 103.000489) (width 0.25) (layer "B.Cu") (net 4))
   (segment (start 95.612511 106.063489) (end 94.488 107.188) (width 0.25) (layer "B.Cu") (net 4))
-  (segment (start 99.187 86.995) (end 99.568 87.376) (width 0.25) (layer "F.Cu") (net 20))
-  (segment (start 95.25 86.995) (end 99.187 86.995) (width 0.25) (layer "F.Cu") (net 20))
-  (segment (start 99.568 87.376) (end 99.568 89.916) (width 0.25) (layer "F.Cu") (net 20))
-  (segment (start 99.568 84.836) (end 99.568 87.376) (width 0.25) (layer "F.Cu") (net 20))
+  (segment (start 99.187 85.979) (end 99.568 86.36) (width 0.25) (layer "F.Cu") (net 20))
+  (segment (start 95.25 86.995) (end 98.933 86.995) (width 0.25) (layer "F.Cu") (net 20))
+  (segment (start 99.568 86.36) (end 99.568 88.9) (width 0.25) (layer "F.Cu") (net 20))
+  (segment (start 98.933 86.995) (end 99.568 86.36) (width 0.25) (layer "F.Cu") (net 20))
+  (segment (start 99.568 83.82) (end 99.568 86.36) (width 0.25) (layer "F.Cu") (net 20))
   (segment (start 103.26 79.375) (end 110.49 79.375) (width 0.2) (layer "F.Cu") (net 21))
   (segment (start 99.775 75.89) (end 103.26 79.375) (width 0.2) (layer "F.Cu") (net 21))
