File: shield/shield.kicad_pcb (KiCad board)
At the start: 2 copper layers, 19.8 x 58.9 mm, 11 parts, among them J2 Battery

Commit message: cleanup
Parts:
- moved C2 13.0 mm to (109.9, 100.6), turned to -90 degrees
- moved J2 11.6 mm to (97.7, 100.6), turned to 0 degrees
- moved C1 4.57 mm to (109.7, 111.8)
- moved R1 4.57 mm to (94.5, 112.3)
- moved R2 4.57 mm to (94.5, 109.2)
- moved HDC1080 3.56 mm to (109.2, 52.8)
- moved Booster1 0.55 mm to (103.3, 99.6), turned to 0 degrees
Routing:
- net Net-(C2-Pad1): track 117.2 -> 110.8 mm
- net GND: track 79.0 -> 84.6 mm
- net Net-(C1-Pad1): track 50.4 -> 55.0 mm
- net Net-(HDC1080-Pad4): track 29.2 -> 31.5 mm
- net +3V3: track 23.8 -> 21.6 mm
- net Net-(HDC1080-Pad3): track 26.4 -> 27.5 mm
Other:
- board size 19.8 x 58.9 mm -> 19.8 x 63.5 mm

Commit message: alpha2 ready
Parts:
- moved Booster1 1.72 mm to (103.3, 97.9)
- moved C2 1.71 mm to (109.9, 98.9)
- moved J2 1.71 mm to (97.7, 98.9)
- moved C1 1.17 mm to (109.7, 110.6)
- moved R1 1.17 mm to (94.5, 111.1)
- moved R2 1.17 mm to (94.5, 108.0)
Routing:
- net Net-(Booster1-Pad1): track 110.8 -> 109.1 mm
- net GND: track 84.6 -> 83.4 mm
- net Net-(C1-Pad1): track 55.0 -> 53.8 mm
- net Net-(HDC1080-Pad4): track 31.5 -> 32.5 mm
