File: shield/shield.kicad_sch (KiCad schematic)
At the start: 12 parts, among them J1 Booster, J2 Battery, P1 Digital, P2 COM, P3 ADC, P4 Analog, P5 ADC, U1 RFM69HW

Commit message: pre holiday commit
Parts:
- removed P1: Digital, Socket_Arduino_Pro_Mini:Socket_Strip_Arduino_1x12, symbol Connector_Generic:Conn_01x12
- removed P2: COM, Socket_Arduino_Pro_Mini:Socket_Strip_Arduino_1x06, symbol Connector_Generic:Conn_01x06
- removed P3, P5: ADC, Socket_Arduino_Pro_Mini:Socket_Strip_Arduino_1x02, symbol Connector_Generic:Conn_01x02
- removed P4: Analog, Socket_Arduino_Pro_Mini:Socket_Strip_Arduino_1x12, symbol Connector_Generic:Conn_01x12
- removed U1: RFM69HW, RF_Module:HOPERF_RFM69HW, symbol RF_Module:RFM69HW
- added J3: SCL Breakout, Connector_PinHeader_2.54mm:PinHeader_1x02_P2.54mm_Vertical, symbol Connector:Conn_01x02_Female
- added J4: SDA Breakout, Connector_PinHeader_2.54mm:PinHeader_1x02_P2.54mm_Vertical, symbol Connector:Conn_01x02_Female
- added ProMini1: rfmshield_pro_mini_pins, footprints:pro_mini_rfmshield, symbol MySymbols:rfmshield_pro_mini_pins
- added RFM69HW1: RFM69HW, RF_Module:HOPERF_RFM69HW, symbol RF_Module:RFM69HW
- C1, C2: footprint Capacitor_THT:C_Rect_L7.0mm_W3.5mm_P2.50mm_P5.00mm -> Capacitor_THT:CP_Radial_D6.3mm_P2.50mm
- J1: value Booster -> Booster Pins; footprint Connector_PinHeader_2.54mm:PinHeader_1x02_P2.54mm_Horizontal -> Connector_PinHeader_2.54mm:PinHeader_1x03_P2.54mm_Vertical
- J2: footprint Connector_PinHeader_2.54mm:PinHeader_1x03_P2.54mm_Horizontal -> Connector_PinHeader_2.54mm:PinHeader_1x02_P2.54mm_Vertical
Connections:
- net GND: now also ProMini1.GND1, RFM69HW1.11 (GND), RFM69HW1.9 (GND)
- net at C2.1, J1.1 (Pin_1): now also ProMini1.VCC, RFM69HW1.8 (3.3V)
- net + renamed +3V3
- net A0: no longer names the net of C1.1, R1.2, R2.1
- net A0: now also ProMini1.VolDiv
- new net: ProMini1.DI00, RFM69HW1.2 (DIO0)
- new net: ProMini1.MISO, RFM69HW1.13 (MISO)
- new net: ProMini1.MOSI, RFM69HW1.14 (MOSI)
- new net: ProMini1.NSS, RFM69HW1.15 (NSS)
- new net: ProMini1.SCK, RFM69HW1.12 (SCK)
- new net: J3.1 (Pin_1), J3.2 (Pin_2), ProMini1.SCL
- new net: J4.1 (Pin_1), J4.2 (Pin_2), ProMini1.SDA
Other:
- note removed: "1"

Commit message: v1-pre renice
Parts:
- removed J3: SCL Breakout, Connector_PinHeader_2.54mm:PinHeader_1x02_P2.54mm_Vertical, symbol Connector:Conn_01x02_Female
- removed J4: SDA Breakout, Connector_PinHeader_2.54mm:PinHeader_1x02_P2.54mm_Vertical, symbol Connector:Conn_01x02_Female
- added J3: Conn_01x03_Female, Connector_PinHeader_2.54mm:PinHeader_1x03_P2.54mm_Vertical, symbol Connector:Conn_01x03_Female
Connections:
- net at ProMini1.GND2: now also J3.1 (Pin_1), J3.2 (Pin_2), J3.3 (Pin_3)
Changed lines of the file:
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@@
   (junction (at 110.49 129.54) (diameter 0) (color 0 0 0 0)
   )
+  (junction (at 133.35 81.28) (diameter 0) (color 0 0 0 0)
+  )
+  (junction (at 133.35 83.82) (diameter 0) (color 0 0 0 0)
+  )
   (junction (at 223.52 124.46) (diameter 0) (color 0 0 0 0)
   )
   (junction (at 68.58 118.11) (diameter 0) (color 0 0 0 0)
   )
-  (junction (at 138.43 93.98) (diameter 0) (color 0 0 0 0)
-  )
   (junction (at 125.73 57.15) (diameter 0) (color 0 0 0 0)
   )
@@
   (junction (at 71.12 132.08) (diameter 0) (color 0 0 0 0)
   )
-  (junction (at 139.7 85.09) (diameter 0) (color 0 0 0 0)
-  )
   (junction (at 113.03 132.08) (diameter 0) (color 0 0 0 0)
   )
   (junction (at 110.49 128.27) (diameter 0) (color 0 0 0 0)
   )
+  (wire (pts (xy 133.35 83.82) (xy 133.35 86.36))
+    (stroke (width 0) (type default) (color 0 0 0 0))
+  )
   (wire (pts (xy 233.68 133.35) (xy 233.68 148.59))
-    (stroke (width 0) (type default) (color 0 0 0 0))
-  )
-  (wire (pts (xy 139.7 85.09) (xy 139.7 87.63))
     (stroke (width 0) (type default) (color 0 0 0 0))
   )
@@
     (stroke (width 0) (type default) (color 0 0 0 0))
   )
+  (wire (pts (xy 133.35 81.28) (xy 133.35 83.82))
+    (stroke (width 0) (type default) (color 0 0 0 0))
+  )
   (wire (pts (xy 125.73 72.39) (xy 219.71 72.39))
     (stroke (width 0) (type default) (color 0 0 0 0))
@@
     (stroke (width 0) (type default) (color 0 0 0 0))
   )
-  (wire (pts (xy 125.73 59.69) (xy 138.43 59.69))
-    (stroke (width 0) (type default) (color 0 0 0 0))
-  )
   (wire (pts (xy 125.73 57.15) (xy 209.55 57.15))
-    (stroke (width 0) (type default) (color 0 0 0 0))
-  )
-  (wire (pts (xy 138.43 93.98) (xy 138.43 96.52))
     (stroke (width 0) (type default) (color 0 0 0 0))
   )
@@
     (stroke (width 0) (type default) (color 0 0 0 0))
   )
+  (wire (pts (xy 133.35 54.61) (xy 133.35 81.28))
+    (stroke (width 0) (type default) (color 0 0 0 0))
+  )
   (wire (pts (xy 234.95 21.59) (xy 234.95 36.83))
+    (stroke (width 0) (type default) (color 0 0 0 0))
+  )
+  (wire (pts (xy 125.73 54.61) (xy 133.35 54.61))
     (stroke (width 0) (type default) (color 0 0 0 0))
   )
@@
     (stroke (width 0) (type default) (color 255 0 0 1))
   )
-  (wire (pts (xy 125.73 62.23) (xy 139.7 62.23))
-    (stroke (width 0) (type default) (color 0 0 0 0))
-  )
-  (wire (pts (xy 139.7 62.23) (xy 139.7 85.09))
-    (stroke (width 0) (type default) (color 0 0 0 0))
-  )
   (wire (pts (xy 125.73 46.99) (xy 201.93 46.99))
-    (stroke (width 0) (type default) (color 0 0 0 0))
-  )
-  (wire (pts (xy 138.43 59.69) (xy 138.43 93.98))
     (stroke (width 0) (type default) (color 0 0 0 0))
   )
@@
     )
     (pin "1")
+  )
+  (symbol (lib_id "Connector:Conn_01x03_Female") (at 138.43 83.82 0) (unit 1)
+    (in_bom yes) (on_board yes) (fields_autoplaced)
+    (property "Reference" "J3" (id 0) (at 139.7 82.5499 0)
+      (effects (font (size 1.27 1.27)) (justify left))
+    )
+    (property "Value" "Conn_01x03_Female" (id 1) (at 139.7 85.0899 0)
+      (effects (font (size 1.27 1.27)) (justify left))
+    )
+    (property "Footprint" "Connector_PinHeader_2.54mm:PinHeader_1x03_P2.54mm_Vertical" (id 2) (at 138.43 83.82 0)
+      (effects (font (size 1.27 1.27)) hide)
+    )
+    (property "Datasheet" "~" (id 3) (at 138.43 83.82 0)
+      (effects (font (size 1.27 1.27)) hide)
+    )
+    (pin "1")
+    (pin "2")
+    (pin "3")
   )
   (symbol (lib_id "MySymbols:rfmshield_pro_mini_pins") (at 120.65 52.07 180) (unit 1)
@@
       (effects (font (size 1.27 1.27)) hide)
     )
+    (pin "1")
+    (pin "18")
+    (pin "19")
+    (pin "2")
+    (pin "20")
+    (pin "22")
+    (pin "3")
+    (pin "DI00")
+    (pin "GND1")
+    (pin "GND2")
+    (pin "MISO")
+    (pin "MOSI")
     (pin "NSS")
     (pin "RAW")
-    (pin "DI00")
-    (pin "GND1")
-    (pin "18")
-    (pin "19")
-    (pin "20")
-    (pin "22")
-    (pin "1")
-    (pin "2")
-    (pin "3")
-    (pin "MOSI")
-    (pin "MISO")
     (pin "SCK")
+    (pin "SCL")
+    (pin "SDA")
+    (pin "VCC")
     (pin "VolDiv")
-    (pin "SDA")
-    (pin "SCL")
-    (pin "VCC")
-    (pin "GND2")
   )
   (symbol (lib_id "RF_Module:RFM69HW") (at 222.25 39.37 90) (unit 1)
@@
     (pin "3")
   )
-  (symbol (lib_id "Connector:Conn_01x02_Female") (at 144.78 85.09 0) (unit 1)
-    (in_bom yes) (on_board yes) (fields_autoplaced)
-    (property "Reference" "J4" (id 0) (at 146.05 85.0899 0)
-      (effects (font (size 1.27 1.27)) (justify left))
-    )
-    (property "Value" "SDA Breakout" (id 1) (at 146.05 87.6299 0)
-      (effects (font (size 1.27 1.27)) (justify left))
-    )
-    (property "Footprint" "Connector_PinHeader_2.54mm:PinHeader_1x02_P2.54mm_Vertical" (id 2) (at 144.78 85.09 0)
-      (effects (font (size 1.27 1.27)) hide)
-    )
-    (property "Datasheet" "~" (id 3) (at 144.78 85.09 0)
-      (effects (font (size 1.27 1.27)) hide)
-    )
-    (pin "1")
-    (pin "2")
-  )
-  (symbol (lib_id "Connector:Conn_01x02_Female") (at 143.51 93.98 0) (unit 1)
-    (in_bom yes) (on_board yes) (fields_autoplaced)
-    (property "Reference" "J3" (id 0) (at 144.78 93.9799 0)
-      (effects (font (size 1.27 1.27)) (justify left))
-    )
-    (property "Value" "SCL Breakout" (id 1) (at 144.78 96.5199 0)
-      (effects (font (size 1.27 1.27)) (justify left))
-    )
-    (property "Footprint" "Connector_PinHeader_2.54mm:PinHeader_1x02_P2.54mm_Vertical" (id 2) (at 143.51 93.98 0)
-      (effects (font (size 1.27 1.27)) hide)
-    )
-    (property "Datasheet" "~" (id 3) (at 143.51 93.98 0)
-      (effects (font (size 1.27 1.27)) hide)
-    )
-    (pin "1")
-    (pin "2")
-  )
   (sheet_instances
     (path "/" (page "1"))
@@
       (reference "J2") (unit 1) (value "Battery") (footprint "Connector_PinHeader_2.54mm:PinHeader_1x02_P2.54mm_Vertical")
     )
-    (path "/ff49efdb-860f-487a-8a24-62300e7a5c79"
-      (reference "J3") (unit 1) (value "SCL Breakout") (footprint "Connector_PinHeader_2.54mm:PinHeader_1x02_P2.54mm_Vertical")
-    )
-    (path "/f746ed1d-6e4f-45c6-bbb9-436542e6ecf2"
-      (reference "J4") (unit 1) (value "SDA Breakout") (footprint "Connector_PinHeader_2.54mm:PinHeader_1x02_P2.54mm_Vertical")
+    (path "/6ef5f8e0-5c2d-4349-9162-179c7c438d89"
+      (reference "J3") (unit 1) (value "Conn_01x03_Female") (footprint "Connector_PinHeader_2.54mm:PinHeader_1x03_P2.54mm_Vertical")
     )
     (path "/a08c2c81-3e22-4b74-ac3d-76da4486ca80"

Commit message: version v1alpha, sent to jclpcb
Parts:
- added HDC1080: Conn_01x04_Female, Connector_PinHeader_2.54mm:PinHeader_1x04_P2.54mm_Vertical, symbol Connector:Conn_01x04_Female
Connections:
- net GND: now also HDC1080.1 (Pin_1)
- net at ProMini1.SCL: now also HDC1080.4 (Pin_4)
- net at ProMini1.SDA: now also HDC1080.3 (Pin_3)
- net at C2.1, J1.1 (Pin_1), ProMini1.VCC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: now also HDC1080.2 (Pin_2)
Changed lines of the file:
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@@
   (junction (at 223.52 148.59) (diameter 0) (color 0 0 0 0)
   )
+  (junction (at 68.58 57.15) (diameter 0) (color 0 0 0 0)
+  )
   (junction (at 71.12 132.08) (diameter 0) (color 0 0 0 0)
   )
+  (junction (at 58.42 46.99) (diameter 0) (color 0 0 0 0)
+  )
   (junction (at 113.03 132.08) (diameter 0) (color 0 0 0 0)
   )
@@
   )
   (wire (pts (xy 233.68 133.35) (xy 233.68 148.59))
+    (stroke (width 0) (type default) (color 0 0 0 0))
+  )
+  (wire (pts (xy 66.04 33.02) (xy 63.5 33.02))
+    (stroke (width 0) (type default) (color 0 0 0 0))
+  )
+  (wire (pts (xy 114.3 59.69) (xy 125.73 59.69))
     (stroke (width 0) (type default) (color 0 0 0 0))
   )
@@
     (stroke (width 0) (type default) (color 255 0 0 1))
   )
+  (wire (pts (xy 58.42 46.99) (xy 58.42 132.08))
+    (stroke (width 0) (type default) (color 0 0 0 0))
+  )
   (wire (pts (xy 125.73 69.85) (xy 217.17 69.85))
     (stroke (width 0) (type default) (color 0 0 0 0))
   )
   (wire (pts (xy 71.12 132.08) (xy 113.03 132.08))
+    (stroke (width 0) (type default) (color 0 0 0 0))
+  )
+  (wire (pts (xy 114.3 38.1) (xy 114.3 59.69))
     (stroke (width 0) (type default) (color 0 0 0 0))
   )
@@
     (stroke (width 0) (type default) (color 0 0 0 0))
   )
-  (wire (pts (xy 125.73 57.15) (xy 68.58 57.15))
+  (wire (pts (xy 68.58 57.15) (xy 125.73 57.15))
     (stroke (width 0) (type default) (color 0 0 0 0))
   )
@@
     (stroke (width 0) (type default) (color 0 0 0 0))
   )
+  (wire (pts (xy 106.68 62.23) (xy 125.73 62.23))
+    (stroke (width 0) (type default) (color 0 0 0 0))
+  )
   (wire (pts (xy 52.07 135.89) (xy 52.07 142.24))
     (stroke (width 0) (type default) (color 0 0 0 0))
@@
     (stroke (width 0) (type default) (color 0 0 0 0))
   )
+  (wire (pts (xy 66.04 35.56) (xy 106.68 35.56))
+    (stroke (width 0) (type default) (color 0 0 0 0))
+  )
   (wire (pts (xy 133.35 54.61) (xy 133.35 81.28))
+    (stroke (width 0) (type default) (color 0 0 0 0))
+  )
+  (wire (pts (xy 66.04 30.48) (xy 58.42 30.48))
     (stroke (width 0) (type default) (color 0 0 0 0))
   )
@@
     (stroke (width 0) (type default) (color 0 0 0 0))
   )
-  (wire (pts (xy 58.42 46.99) (xy 58.42 132.08))
+  (wire (pts (xy 58.42 30.48) (xy 58.42 46.99))
+    (stroke (width 0) (type default) (color 0 0 0 0))
+  )
+  (wire (pts (xy 63.5 33.02) (xy 63.5 57.15))
     (stroke (width 0) (type default) (color 0 0 0 0))
   )
@@
     (stroke (width 0) (type default) (color 0 0 0 0))
   )
+  (wire (pts (xy 66.04 38.1) (xy 114.3 38.1))
+    (stroke (width 0) (type default) (color 0 0 0 0))
+  )
   (wire (pts (xy 113.03 132.08) (xy 113.03 148.59))
     (stroke (width 0) (type default) (color 0 0 0 0))
@@
     (stroke (width 0) (type default) (color 0 0 0 0))
   )
-  (wire (pts (xy 125.73 46.99) (xy 58.42 46.99))
+  (wire (pts (xy 58.42 46.99) (xy 125.73 46.99))
     (stroke (width 0) (type default) (color 0 0 0 0))
   )
@@
   )
   (wire (pts (xy 201.93 46.99) (xy 201.93 21.59))
+    (stroke (width 0) (type default) (color 0 0 0 0))
+  )
+  (wire (pts (xy 106.68 35.56) (xy 106.68 62.23))
+    (stroke (width 0) (type default) (color 0 0 0 0))
+  )
+  (wire (pts (xy 63.5 57.15) (xy 68.58 57.15))
     (stroke (width 0) (type default) (color 0 0 0 0))
   )
@@
     (pin "9")
   )
+  (symbol (lib_id "Connector:Conn_01x04_Female") (at 71.12 33.02 0) (unit 1)
+    (in_bom yes) (on_board yes) (fields_autoplaced)
+    (property "Reference" "HDC1080" (id 0) (at 72.39 33.0199 0)
+      (effects (font (size 1.27 1.27)) (justify left))
+    )
+    (property "Value" "Conn_01x04_Female" (id 1) (at 72.39 35.5599 0)
+      (effects (font (size 1.27 1.27)) (justify left))
+    )
+    (property "Footprint" "Connector_PinHeader_2.54mm:PinHeader_1x04_P2.54mm_Vertical" (id 2) (at 71.12 33.02 0)
+      (effects (font (size 1.27 1.27)) hide)
+    )
+    (property "Datasheet" "~" (id 3) (at 71.12 33.02 0)
+      (effects (font (size 1.27 1.27)) hide)
+    )
+    (pin "1")
+    (pin "2")
+    (pin "3")
+    (pin "4")
+  )
   (symbol (lib_id "Connector:Conn_01x02_Female") (at 110.49 123.19 90) (unit 1)
     (in_bom yes) (on_board yes)
@@
       (reference "C2") (unit 1) (value "C Booster") (footprint "Capacitor_THT:CP_Radial_D6.3mm_P2.50mm")
     )
+    (path "/b16db6aa-eff9-4560-94eb-8f1df0edf71a"
+      (reference "HDC1080") (unit 1) (value "Conn_01x04_Female") (footprint "Connector_PinHeader_2.54mm:PinHeader_1x04_P2.54mm_Vertical")
+    )
     (path "/f022c12c-8ce1-4cb0-9f5f-a1e5ee7d0ba0"

Commit message: pics
Parts:
- added Extra3v3: Conn_01x03_Female, Connector_PinHeader_2.54mm:PinHeader_1x03_P2.54mm_Vertical, symbol Connector:Conn_01x03_Female
- HDC1080: value Conn_01x04_Female -> HDC1080
- renumbered J1 to Booster1, J3 to ExtraGND1
Connections:
- net at Booster1.1 (Pin_1), C2.1, HDC1080.2 (Pin_2)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: now also Extra3v3.1 (Pin_1), Extra3v3.2 (Pin_2), Extra3v3.3 (Pin_3)
Changed lines of the file:
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@@
   (junction (at 125.73 57.15) (diameter 0) (color 0 0 0 0)
   )
+  (junction (at 73.66 91.44) (diameter 0) (color 0 0 0 0)
+  )
   (junction (at 113.03 128.27) (diameter 0) (color 0 0 0 0)
   )
@@
   (junction (at 71.12 132.08) (diameter 0) (color 0 0 0 0)
   )
+  (junction (at 68.58 91.44) (diameter 0) (color 0 0 0 0)
+  )
   (junction (at 58.42 46.99) (diameter 0) (color 0 0 0 0)
   )
@@
     (stroke (width 0) (type default) (color 0 0 0 0))
   )
+  (wire (pts (xy 68.58 91.44) (xy 68.58 118.11))
+    (stroke (width 0) (type default) (color 255 0 0 1))
+  )
   (wire (pts (xy 233.68 133.35) (xy 233.68 148.59))
     (stroke (width 0) (type default) (color 0 0 0 0))
@@
     (stroke (width 0) (type default) (color 0 0 0 0))
   )
-  (wire (pts (xy 68.58 57.15) (xy 68.58 118.11))
+  (wire (pts (xy 68.58 57.15) (xy 68.58 91.44))
     (stroke (width 0) (type default) (color 255 0 0 1))
   )
@@
     (stroke (width 0) (type default) (color 0 0 0 0))
   )
+  (wire (pts (xy 68.58 91.44) (xy 73.66 91.44))
+    (stroke (width 0) (type default) (color 0 0 0 0))
+  )
   (wire (pts (xy 58.42 132.08) (xy 71.12 132.08))
     (stroke (width 0) (type default) (color 0 0 0 0))
@@
     (stroke (width 0) (type default) (color 255 0 0 1))
   )
+  (wire (pts (xy 73.66 88.9) (xy 73.66 91.44))
+    (stroke (width 0) (type default) (color 0 0 0 0))
+  )
+  (wire (pts (xy 73.66 91.44) (xy 73.66 93.98))
+    (stroke (width 0) (type default) (color 0 0 0 0))
+  )
   (wire (pts (xy 125.73 46.99) (xy 201.93 46.99))
     (stroke (width 0) (type default) (color 0 0 0 0))
@@
     (effects (font (size 1.27 1.27)) (justify left bottom))
   )
+  (symbol (lib_id "Connector:Conn_01x03_Female") (at 78.74 91.44 0) (unit 1)
+    (in_bom yes) (on_board yes) (fields_autoplaced)
+    (property "Reference" "Extra3v3" (id 0) (at 80.01 90.1699 0)
+      (effects (font (size 1.27 1.27)) (justify left))
+    )
+    (property "Value" "Conn_01x03_Female" (id 1) (at 80.01 92.7099 0)
+      (effects (font (size 1.27 1.27)) (justify left))
+    )
+    (property "Footprint" "Connector_PinHeader_2.54mm:PinHeader_1x03_P2.54mm_Vertical" (id 2) (at 78.74 91.44 0)
+      (effects (font (size 1.27 1.27)) hide)
+    )
+    (property "Datasheet" "~" (id 3) (at 78.74 91.44 0)
+      (effects (font (size 1.27 1.27)) hide)
+    )
+    (pin "1")
+    (pin "2")
+    (pin "3")
+  )
   (symbol (lib_id "Device:C") (at 223.52 144.78 0) (unit 1)
     (in_bom yes) (on_board yes) (fields_autoplaced)
@@
   (symbol (lib_id "Connector:Conn_01x03_Female") (at 138.43 83.82 0) (unit 1)
     (in_bom yes) (on_board yes) (fields_autoplaced)
-    (property "Reference" "J3" (id 0) (at 139.7 82.5499 0)
+    (property "Reference" "ExtraGND1" (id 0) (at 139.7 82.5499 0)
       (effects (font (size 1.27 1.27)) (justify left))
     )
@@
       (effects (font (size 1.27 1.27)) (justify left))
     )
-    (property "Value" "Conn_01x04_Female" (id 1) (at 72.39 35.5599 0)
+    (property "Value" "HDC1080" (id 1) (at 72.39 35.5599 0)
       (effects (font (size 1.27 1.27)) (justify left))
     )
@@
   (symbol (lib_id "Connector:Conn_01x03_Female") (at 71.12 113.03 90) (unit 1)
     (in_bom yes) (on_board yes) (fields_autoplaced)
-    (property "Reference" "J1" (id 0) (at 71.12 107.95 90))
+    (property "Reference" "Booster1" (id 0) (at 71.12 107.95 90))
     (property "Value" "Booster Pins" (id 1) (at 71.12 110.49 90))
     (property "Footprint" "Connector_PinHeader_2.54mm:PinHeader_1x03_P2.54mm_Vertical" (id 2) (at 71.12 113.03 0)
@@
       (reference "#PWR0102") (unit 1) (value "GND") (footprint "")
     )
+    (path "/f022c12c-8ce1-4cb0-9f5f-a1e5ee7d0ba0"
+      (reference "Booster1") (unit 1) (value "Booster Pins") (footprint "Connector_PinHeader_2.54mm:PinHeader_1x03_P2.54mm_Vertical")
+    )
     (path "/386ab483-3160-4f1e-9c93-fbcb1e235786"
       (reference "C1") (unit 1) (value "C Voltage Divider") (footprint "Capacitor_THT:CP_Radial_D6.3mm_P2.50mm")
@@
       (reference "C2") (unit 1) (value "C Booster") (footprint "Capacitor_THT:CP_Radial_D6.3mm_P2.50mm")
     )
+    (path "/077985bd-c8a6-43b8-af30-1141a8334306"
+      (reference "Extra3v3") (unit 1) (value "Conn_01x03_Female") (footprint "Connector_PinHeader_2.54mm:PinHeader_1x03_P2.54mm_Vertical")
+    )
+    (path "/6ef5f8e0-5c2d-4349-9162-179c7c438d89"
+      (reference "ExtraGND1") (unit 1) (value "Conn_01x03_Female") (footprint "Connector_PinHeader_2.54mm:PinHeader_1x03_P2.54mm_Vertical")
+    )
     (path "/b16db6aa-eff9-4560-94eb-8f1df0edf71a"
-      (reference "HDC1080") (unit 1) (value "Conn_01x04_Female") (footprint "Connector_PinHeader_2.54mm:PinHeader_1x04_P2.54mm_Vertical")
-    )
-    (path "/f022c12c-8ce1-4cb0-9f5f-a1e5ee7d0ba0"
-      (reference "J1") (unit 1) (value "Booster Pins") (footprint "Connector_PinHeader_2.54mm:PinHeader_1x03_P2.54mm_Vertical")
+      (reference "HDC1080") (unit 1) (value "HDC1080") (footprint "Connector_PinHeader_2.54mm:PinHeader_1x04_P2.54mm_Vertical")
     )
     (path "/b8790514-1424-44a6-b36e-2e7680815de1"
       (reference "J2") (unit 1) (value "Battery") (footprint "Connector_PinHeader_2.54mm:PinHeader_1x02_P2.54mm_Vertical")
     )
-    (path "/6ef5f8e0-5c2d-4349-9162-179c7c438d89"
-      (reference "J3") (unit 1) (value "Conn_01x03_Female") (footprint "Connector_PinHeader_2.54mm:PinHeader_1x03_P2.54mm_Vertical")
-    )
     (path "/a08c2c81-3e22-4b74-ac3d-76da4486ca80"
